Commit message: Add finger link offsets

File: pal_gripper_description/urdf/gripper.urdf.xacro (robot description, xacro)
@@ -62,5 +62,5 @@
     </inertial>
     <visual>
-      <origin rpy="0 0 3.1415" xyz="0 0 0" />
+      <origin rpy="0 0 3.1415" xyz="0.013 0 0" />
       <geometry>
         <mesh filename="package://pal_gripper_description/meshes/gripper_finger_link.stl" scale="-1 -1 1"/>
@@ -69,5 +69,5 @@
     </visual>
     <collision>
-      <origin rpy="0 0 3.1415" xyz="0.005 0 -0.165" />
+      <origin rpy="0 0 3.1415" xyz="0.018 0 -0.165" />
       <geometry>
         <box size="0.01 0.05 0.11"/>
@@ -100,5 +100,5 @@
     </inertial>
     <visual>
-      <origin rpy="0 0 3.1415" xyz="0 0 0"/>
+      <origin rpy="0 0 3.1415" xyz="-0.013 0 0"/>
       <geometry>
         <mesh filename="package://pal_gripper_description/meshes/gripper_finger_link.stl"/>
@@ -107,5 +107,5 @@
     </visual>
     <collision>
-      <origin rpy="0 0 3.1415" xyz="-0.005 0 -0.165" />
+      <origin rpy="0 0 3.1415" xyz="-0.018 0 -0.165" />
       <geometry>
         <box size="0.01 0.05 0.11"/>
